File: fdm_3dp_thermistor_breakout.kicad_sch (KiCad schematic)
At the start: 8 parts, among them J1 Conn_01x03_Pin, J2 Conn_01x02_Socket

Commit message: parts sourced
Parts:
- C1: MPN1 (none) -> Wurth Elektronik:860130673001; SKU1 (none) -> Distrelec:302-28-156
- J1: MPN1 (none) -> Molex:43650-0315; SKU1 (none) -> Distrelec:144-02-076
- J2: MPN1 (none) -> Molex:43650-0215; SKU1 (none) -> Distrelec:144-02-069
- R1: MPN1 (none) -> Vishay:MBA02040C4701FCT00; SKU1 (none) -> Distrelec:160-59-406
Connections:
- net Thermistor: now reaches C1.1, J1.2 (Pin_2), J2.1 (Pin_1), R1.2
Changed lines of the file:
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@@
     (effects (font (size 1.27 1.27)) (justify left bottom) (href "https://reprap.org/wiki/RAMPS_1.4"))
   )
+  (hierarchical_label "Thermistor" (shape input) (at 120.65 101.6 90) (fields_autoplaced)
+    (effects (font (size 1.27 1.27)) (justify left))
+  )
+  (hierarchical_label "+5V" (shape input) (at 120.65 87.63 90) (fields_autoplaced)
+    (effects (font (size 1.27 1.27)) (justify left))
+  )
+  (hierarchical_label "GND" (shape input) (at 120.65 118.11 90) (fields_autoplaced)
+    (effects (font (size 1.27 1.27)) (justify left))
+  )
   (symbol (lib_id "Mechanical:MountingHole") (at 15.24 194.31 0) (unit 1)
     (in_bom yes) (on_board yes) (dnp no) (fields_autoplaced)
@@
     )
     (instances
-      (project "thermistor"
+      (project "fdm_3dp_thermistor_breakout"
         (path "/c28ea80b-ab5a-400c-b331-afff352bd79f"
           (reference "H4") (unit 1)
@@
       (effects (font (size 1.27 1.27)) hide)
     )
-    (property "Datasheet" "~" (at 149.86 110.49 0)
-      (effects (font (size 1.27 1.27)) hide)
-    )
-    (pin "1")
-    (pin "2")
-    (instances
-      (project "thermistor"
+    (property "Datasheet" "https://octopart.com/datasheet/860130673001-wurth+elektronik-54218090" (at 149.86 110.49 0)
+      (effects (font (size 1.27 1.27)) hide)
+    )
+    (property "MPN1" "Wurth Elektronik:860130673001" (at 149.86 110.49 0)
+      (effects (font (size 1.27 1.27)) hide)
+    )
+    (property "SKU1" "Distrelec:302-28-156" (at 149.86 110.49 0)
+      (effects (font (size 1.27 1.27)) hide)
+    )
+    (pin "1")
+    (pin "2")
+    (instances
+      (project "fdm_3dp_thermistor_breakout"
         (path "/c28ea80b-ab5a-400c-b331-afff352bd79f"
           (reference "C1") (unit 1)
@@
     )
     (instances
-      (project "thermistor"
+      (project "fdm_3dp_thermistor_breakout"
         (path "/c28ea80b-ab5a-400c-b331-afff352bd79f"
           (reference "H3") (unit 1)
@@
       (effects (font (size 1.27 1.27)) hide)
     )
-    (property "Datasheet" "~" (at 190.5 101.6 0)
-      (effects (font (size 1.27 1.27)) hide)
-    )
-    (pin "1")
-    (pin "2")
-    (instances
-      (project "thermistor"
+    (property "Datasheet" "https://octopart.com/datasheet/43650-0215-molex-298121" (at 190.5 101.6 0)
+      (effects (font (size 1.27 1.27)) hide)
+    )
+    (property "MPN1" "Molex:43650-0215" (at 190.5 101.6 0)
+      (effects (font (size 1.27 1.27)) hide)
+    )
+    (property "SKU1" "Distrelec:144-02-069" (at 190.5 101.6 0)
+      (effects (font (size 1.27 1.27)) hide)
+    )
+    (pin "1")
+    (pin "2")
+    (instances
+      (project "fdm_3dp_thermistor_breakout"
         (path "/c28ea80b-ab5a-400c-b331-afff352bd79f"
           (reference "J2") (unit 1)
@@
       (effects (font (size 1.27 1.27)) hide)
     )
-    (property "Datasheet" "~" (at 149.86 95.25 0)
-      (effects (font (size 1.27 1.27)) hide)
-    )
-    (pin "1")
-    (pin "2")
-    (instances
-      (project "thermistor"
+    (property "Datasheet" "https://octopart.com/datasheet/mba02040c4701fct00-vishay-43744265" (at 149.86 95.25 0)
+      (effects (font (size 1.27 1.27)) hide)
+    )
+    (property "SKU1" "Distrelec:160-59-406" (at 149.86 95.25 0)
+      (effects (font (size 1.27 1.27)) hide)
+    )
+    (property "MPN1" "Vishay:MBA02040C4701FCT00" (at 149.86 95.25 0)
+      (effects (font (size 1.27 1.27)) hide)
+    )
+    (pin "1")
+    (pin "2")
+    (instances
+      (project "fdm_3dp_thermistor_breakout"
         (path "/c28ea80b-ab5a-400c-b331-afff352bd79f"
           (reference "R1") (unit 1)
@@
     )
     (instances
-      (project "thermistor"
+      (project "fdm_3dp_thermistor_breakout"
         (path "/c28ea80b-ab5a-400c-b331-afff352bd79f"
           (reference "H1") (unit 1)
@@
     )
     (instances
-      (project "thermistor"
+      (project "fdm_3dp_thermistor_breakout"
         (path "/c28ea80b-ab5a-400c-b331-afff352bd79f"
           (reference "H2") (unit 1)
@@
       (effects (font (size 1.27 1.27)) hide)
     )
+    (property "MPN1" "Molex:43650-0315" (at 106.68 101.6 0)
+      (effects (font (size 1.27 1.27)) hide)
+    )
+    (property "SKU1" "Distrelec:144-02-076" (at 106.68 101.6 0)
+      (effects (font (size 1.27 1.27)) hide)
+    )
     (pin "1")
     (pin "2")
     (pin "3")
     (instances
-      (project "thermistor"
+      (project "fdm_3dp_thermistor_breakout"
         (path "/c28ea80b-ab5a-400c-b331-afff352bd79f"
           (reference "J1") (unit 1)
@@
     (pin "1")
     (instances
-      (project "thermistor"
+      (project "fdm_3dp_thermistor_breakout"
         (path "/c28ea80b-ab5a-400c-b331-afff352bd79f"
           (reference "#PWR01") (unit 1)
@@
     (pin "1")
     (instances
-      (project "thermistor"
+      (project "fdm_3dp_thermistor_breakout"
         (path "/c28ea80b-ab5a-400c-b331-afff352bd79f"
           (reference "#PWR02") (unit 1)
